Commit message: Code used for the video

File: motoman-hydro-devel/motoman_sda10f_support/urdf/sda10f_macro.xacro (robot description, xacro)
@@ -32,4 +32,49 @@
 		</visual>
 	</link>
+    <link name="camera_left">
+		<visual>
+			<geometry>
+				<box size=".11 .025 .035" />
+			</geometry>
+            <material name="pwkl">
+          		<color rgba=".8 .8 1 1"/>
+         	</material>
+		</visual>
+	</link>
+    <joint name="camera_joint_left" type="fixed">
+            <origin rpy="0 0 0" xyz="0 0 .083"/>
+                <parent link="hand_left_palm" />
+                <child link="camera_left" />
+        </joint>
+    <link name="robotiq_hand_wires_left">
+		<visual>
+			<geometry>
+				<box size=".045 .05 .07" />
+			</geometry>
+            <material name="pwkl">
+          		<color rgba=".8 .6 1 1"/>
+         	</material>
+		</visual>
+	</link>
+    <joint name="robotiq_hand_wires_left_joint" type="fixed">
+            <origin rpy="0 0 0" xyz="0.08 -0.02 0.0"/>
+                <parent link="hand_left_palm" />
+                <child link="robotiq_hand_wires_left" />
+    </joint>
+    <link name="robotiq_force_wires_left">
+		<visual>
+			<geometry>
+				<box size=".045 .05 .02" />
+			</geometry>
+            <material name="pwkl">
+          		<color rgba=".8 0 1 1"/>
+         	</material>
+		</visual>
+	</link>
+    <joint name="robotiq_force_wires_left_joint" type="fixed">
+            <origin rpy="0 0 0" xyz="0.09 0 0"/>
+                <parent link="cylinder_hand_left" />
+                <child link="robotiq_force_wires_left" />
+    </joint>
 <!--
 	<link name="ft_sensor_cable_box_left">
@@ -49,10 +94,10 @@
 -->
         <joint name="hand_cylinder_joint_left" type="fixed">
-            <origin rpy="3.14159 0 0" xyz="0 0 0"/>
+            <origin rpy="3.14159 0 3.14159" xyz="0 0 0"/>
                 <parent link="arm_left_link_tool0" />
                 <child link="cylinder_hand_left" />
         </joint>
         <joint name="hand_cylinder_joint_right" type="fixed">
-            <origin rpy="3.14159 0 0" xyz="0 0 -.03125"/>
+            <origin rpy="3.14159 0 3.14159" xyz="0 0 -.03125"/>
                 <parent link="arm_right_link_tool0" />
                 <child link="cylinder_hand_right" />
@@ -63,5 +108,5 @@
 <!--.077475-->
         <joint name="hand_left_joint" type="fixed">
-           <origin rpy="1.57079 0 2.87979" xyz="0 0 0.0797125"/>
+           <origin rpy="1.57079 0 -0.26180" xyz="0 0 0.0797125"/>
                 <parent link="cylinder_hand_left" />
                 <child link="hand_left_palm" />
@@ -76,5 +121,5 @@
         </xacro:s-model_articulated>
         <joint name="hand_right_joint" type="fixed">
-           <origin rpy="1.57079 0 -0.261799" xyz="0 0 0.0797125"/>
+           <origin rpy="1.57079 0 2.87979" xyz="0 0 0.0797125"/>
                 <parent link="cylinder_hand_right" />
                 <child link="hand_right_palm" />

File: robotiq-indigo-devel_custom/robotiq_s_model_visualization/cfg/s-model_articulated_macro.xacro (robot description, xacro)
@@ -23,5 +23,5 @@
 			<collision>
 				<geometry>
-					<mesh filename="package://robotiq_s_model_visualization/meshes/s-model_articulated/collision/palm.STL" />
+					<mesh filename="package://robotiq_s_model_visualization/meshes/s-model_articulated/visual/palm.STL" />
 				</geometry>
 				<material name="yellow">

File: robotiq-indigo-devel_custom/robotiq_s_model_visualization/cfg/s-model_finger_articulated_macro.xacro (robot description, xacro)
@@ -19,5 +19,6 @@
 			</visual>
 			<collision>
-				<origin xyz="-0.0455 0.0414 0.036" rpy="0 3.1416 -1.57"/>
+				<!--<origin xyz="-0.0455 0.0414 0.036" rpy="0 3.1416 -1.57"/>-->
+                <origin xyz="0.020 0 0" rpy="0 0 0"/>
 				<geometry>
 					<mesh filename="package://robotiq_s_model_visualization/meshes/s-model_articulated/collision/link_0.STL" />
